File: Project4-robot_line_follower/Design_PCB/core/core.sch (EAGLE design)
At the start: 23 parts, among them IC1 MCP3008-I_P, IC2 AT24CP, IC4 7402N, M1 ARDUINO-NANO-3.0

Commit message: rename file
Parts:
- removed IC1: MCP3008-I_P, MCP3008-I_P:MCP3008-I_P
- removed IC2: AT24CP, atmel:AT24CP
- removed IC4: 7402N, 74xx-us:7402N
- removed JP1: (no value), pinhead:PINHD-1X4
- added JP3: (no value), pinhead:PINHD-1X11
- added JP5: (no value), pinhead:PINHD-1X6
- added LED2: (no value), led:LED3MM
- added R4, R5: 1K, rcl:R-EU_0207/7
- added T1: BD139, transistor-neu-to92:BD139
- JP4: device pinhead:PINHD-1X16 -> pinhead:PINHD-1X6
- R2: value 4.7K -> 22K
- R3: value 4.7K -> (none); device rcl:R-EU_0207/7 -> pot:TRIM_EU-CA6V
Connections:
- removed net 1A: IC4A.O, JP2.3
- removed net 1B: IC4A.I0, IC4B.O, JP2.4
- removed net 2A: IC4D.O, JP2.5
- removed net 2B: IC4C.O, IC4D.I0, JP2.6
- removed net 5V: C1.+, IC1.VDD, IC1.VREF, IC2.VCC, IC4P.VCC, JP1.2, JP4.15, M1.VIN, R1.2, R2.2, R3.2, U$1.OUT+
- removed net A0: JP4.14, M1.A0
- removed net A10: IC1.CH4, JP4.4
- removed net A11: IC1.CH5, JP4.3
- removed net A12: IC1.CH6, JP4.2
- removed net A13: IC1.CH7, JP4.1
- removed net A8: IC1.CH2, JP4.6
- removed net A9: IC1.CH3, JP4.5
- removed net B5: M1.D4, S4.S, S4.S1
- removed net B6: M1.D9
- removed net CS: IC1.!CS!/SHDN, M1.D10
- removed net DIR1: IC4B.I1, M1.D7
- removed net DIR2: IC4C.I1, M1.D8
- removed net MISO: IC1.DOUT, M1.D12/MISO
- removed net MOSI: IC1.DIN, M1.D11/MOSI
- removed net N$4: JP2.2, S81.P
- removed net PWM1: IC4A.I1, IC4B.I0, M1.D5
- removed net PWM2: IC4C.I0, IC4D.I1, M1.D6
- removed net SCK: IC1.CLK, M1.D13/SCK
- removed net SCL: IC2.SCL, JP1.4, M1.A5, R3.1
- removed net SDA: IC2.SDA, JP1.3, M1.A4, R2.1
- new net 12VM: JP2.2, R2.1, S81.P
- new net 5VIN: C1.+, JP3.2, JP4.2, JP5.5, M1.VIN, R1.2, R3.E, R5.2, U$1.OUT+
- new net D4: JP5.1, M1.D10
- new net D5: JP5.2, M1.D9
- new net D6: JP5.3, M1.D8
- new net D7: JP5.4, M1.D7
- new net E: JP4.6, M1.D12/MISO
- new net L: JP3.3, R5.1, T1.C
- new net N$6: LED2.A, R2.2
- new net N$7: R4.1, T1.B
- new net N$8: JP4.3, R3.S
- new net N$9: M1.5V
- new net PWM1A: JP2.6, M1.D6
- new net PWM1B: JP2.5, M1.D5
- new net PWM2A: JP2.4, M1.D11/MOSI
- new net PWM2B: JP2.3, M1.D3
- new net R: JP3.4, M1.A0, R4.2
- new net RS: JP4.4, M1.D13/SCK
- net A1: now also JP3.5; no longer JP4.13
- net A2: now also JP3.6; no longer JP4.12
- net A3: now also JP3.7; no longer JP4.11
- net A4: now also JP3.8, M1.A4; no longer JP4.10, M1.A6
- net A5: now also JP3.9, M1.A5; no longer JP4.9, M1.A7
- net A6: now also JP3.10, M1.A6; no longer IC1.CH0, JP4.8
- net A7: now also JP3.11, M1.A7; no longer IC1.CH1, JP4.7
- net B1: now also S1.S, S1.S1
- net B2: now also S2.S, S2.S1; no longer S1.S, S1.S1
- net B3: now also S3.S, S3.S1; no longer S2.S, S2.S1
- net B4: now also M1.D4, S4.S, S4.S1; no longer M1.D3, S3.S, S3.S1
- net GND: now also JP3.1, JP4.1, JP4.5, JP5.6, LED2.C, R3.A, T1.E; no longer IC1.AGND, IC1.DGND, IC2.A0, IC2.A1, IC2.A2, IC2.GND, IC2.WP, IC4P.GND, JP1.1, JP4.16
Other:
- moved on the sheet: R2
